Commit message: Added DH-Parameters and Forward Kinematics

File: lbr_fri_ros2_stack/lbr_description/urdf/iiwa14/iiwa14_description.xacro (robot description, xacro)
@@ -42,5 +42,5 @@
         </link>
         <joint name="A1" type="revolute">
-            <origin rpy="0 0 0" xyz="0.0 0.0 0.1475" />
+            <origin rpy="0 0 0" xyz="0.0 0.0 0.15" />
             <parent link="link_0" />
             <child link="link_1" />
